File: betadisk/beta128_r0.3.sch (KiCad schematic (older format))
At the start: 85 parts, among them J1 ZX_Spectrum_Connector_GENERIC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, J2 Conn_02x17_Odd_Even, Q1 BC639, SW1 SW_DIP_x02, U10 74LS174, U11 74LS367, U12 FDC_MB8877, U13 74LS14, U14 74LS139, U15 74LS06, U16 74LS74, U17 74LS161, U18 74LS161, U19 74LS00, U21 L7805, U22 GAL22V10, U3 W27C512, U4 74LS32, U6 74LS30, U7 74LS123, U8 74LS74, U9 74LS07, U99 74LS245, Y1 8.000Mhz

Commit message: update on libs
Parts:
- C5: symbol dos_5-0x-eagle-import:C-EU025-030X050 -> Device:C
- J1: symbol ALEA:ZX_Spectrum_Connector_GENERIC_SORTED -> 8bits:ZX_Spectrum_Connector_GENERIC_SORTED
- R1, R18, R2, R21, R22, R3, R5: symbol dos_5-0x-eagle-import:R-EU_0207_10 -> Device:R
- U12: symbol ALEA:FDC_MB8877 -> 8bits:FDC_MB8877
- U22: symbol ALEA:GAL22V10 -> 8bits:GAL22V10
- U3: symbol ALEA:W27C512 -> 8bits:W27C512
Connections:
- wire segments 576 -> 579
Changed lines of the file:
@@
 Connection ~ 11150 8450
 Connection ~ 11150 9450
-Connection ~ 11350 4000
 Connection ~ 11350 4800
 Connection ~ 11600 4800
@@
 Connection ~ 24200 5700
 Connection ~ 24550 9350
-Connection ~ 25150 5300
 Connection ~ 25900 9550
 Connection ~ 26400 8550
@@
 Connection ~ 27850 7300
 Connection ~ 28500 8850
+Connection ~ 11350 4000
+Connection ~ 25150 5300
 NoConn ~ 1600 1500
 NoConn ~ 1600 1600
@@
 	21250 7350 21350 7250
 Wire Wire Line
-	625  2200 625  2300
+	650  2200 650  2400
 Wire Wire Line
 	850  1800 1600 1800
@@
 	1325 2100 1600 2100
 Wire Wire Line
-	1325 2200 625  2200
+	1325 2200 650  2200
 Wire Wire Line
 	1375 5550 1375 5650
@@
 	7650 2450 7650 2350
 Wire Wire Line
-	7850 1850 7850 1900
+	7850 1850 7850 1950
 Wire Wire Line
-	7850 2300 7850 2350
+	7850 2250 7850 2350
 Wire Wire Line
 	7850 2350 8450 2350
@@
 	9850 6500 10600 6500
 Wire Wire Line
-	9950 1050 9950 1100
+	9950 1050 9950 1150
 Wire Wire Line
-	9950 1500 9950 1550
+	9950 1450 9950 1550
 Wire Wire Line
 	9950 1550 9950 1600
@@
 	11350 2050 11300 2050
 Wire Wire Line
-	11350 2050 11350 3600
+	11350 2050 11350 3650
+Wire Wire Line
+	11350 3950 11350 4000
 Wire Wire Line
 	11350 4000 11800 4000
 Wire Wire Line
-	11350 4300 11350 4350
+	11350 4300 11350 4400
 Wire Wire Line
-	11350 4750 11350 4800
+	11350 4700 11350 4800
 Wire Wire Line
 	11350 4800 11100 4800
@@
 	22250 8200 22100 8200
 Wire Wire Line
-	22400 8200 22400 8250
+	22400 8200 22400 8300
+Wire Wire Line
+	22400 8600 22400 8650
 Wire Wire Line
 	22400 8650 22350 8650
@@
 	23650 9550 24600 9550
 Wire Wire Line
-	23750 8000 23750 7950
+	23750 7950 23750 8050
 Wire Wire Line
-	23750 8400 23750 8450
+	23750 8350 23750 8450
 Wire Wire Line
 	23750 8450 23800 8450
@@
 	25050 5700 24200 5700
 Wire Wire Line
+	25100 5300 25150 5300
+Wire Wire Line
 	25150 3000 25150 3700
 Wire Wire Line
-	25150 4900 25150 4850
+	25150 4850 25150 4950
 Wire Wire Line
-	25150 5300 25100 5300
+	25150 5250 25150 5300
+Wire Wire Line
+	25150 5300 25300 5300
 Wire Wire Line
 	25150 6700 27350 6700
@@
 	25300 4100 25350 4100
 Wire Wire Line
-	25300 5300 25150 5300
-Wire Wire Line
 	25350 3000 25150 3000
 Wire Wire Line
@@
 	3700 1600 3700 1800
 Wire Bus Line
-	3700 1800 3700 1900
+	3700 1800 3700 2000
 Wire Bus Line
-	3700 1900 3700 2100
+	3700 2000 3700 2200
 Wire Bus Line
-	3700 2100 3700 2300
+	3700 2200 3700 2400
 Wire Bus Line
-	3700 2300 3700 2500
+	3700 2400 3700 2500
 Wire Bus Line
 	3700 2500 3700 2700
@@
 	3700 2900 3700 3000
 Wire Bus Line
-	3700 3200 3700 3300
+	3700 3200 3700 3400
 Wire Bus Line
-	3700 3300 3700 3500
+	3700 3400 3700 3500
 Wire Bus Line
-	3700 3500 3700 3600
+	3700 3500 3700 3700
 Wire Bus Line
-	3700 3600 3700 3800
+	3700 3700 3700 3900
 Wire Bus Line
-	3700 3800 3700 4550
+	3700 3900 3700 4650
 Wire Bus Line
-	3700 4550 3700 4750
+	3700 4650 3700 4850
 Wire Bus Line
-	3700 4750 3700 4950
+	3700 4850 3700 4950
 Wire Bus Line
 	3700 4950 3700 5150
@@
 	5500 2800 5500 4650
 Wire Bus Line
-	5500 4650 5500 4750
+	5500 4650 5500 4850
 Wire Bus Line
-	5500 4750 5500 4950
+	5500 4850 5500 5050
 Wire Bus Line
-	5500 4950 5500 5150
+	5500 5050 5500 5250
 Wire Bus Line
-	5500 5150 5500 5600
+	5500 5250 5500 5600
 Wire Bus Line
-	6450 1000 6450 1500
+	6450 1000 6450 1150
 Wire Bus Line
-	6450 1500 6450 1700
+	6450 1150 6450 1600
+Wire Bus Line
+	6450 1600 6450 1700
 Wire Bus Line
 	6450 1700 6450 1900
 Wire Bus Line
-	6450 1900 6450 2100
+	6450 1900 6450 2000
 Wire Bus Line
-	6450 2100 6450 2800
+	6450 2000 6450 2800
 Wire Bus Line
 	6450 2800 5500 2800
@@
 $EndComp
 $Comp
+L power:GND #GND010
+U 1 1 845C69E3
+P 650 2400
+F 0 "#GND010" H 650 2400 50  0001 C CNN
+F 1 "GND" H 575 2200 60  0000 L BNN
+F 2 "" H 650 2400 50  0001 C CNN
+F 3 "" H 650 2400 50  0001 C CNN
+	1    650  2400
+	1    0    0    -1
+$EndComp
+$Comp
 L power:GND #PWR021
 U 1 1 5B4CC0A2
@@
 $EndComp
 $Comp
-L dos_5-0x-eagle-import:GND #GND010
-U 1 1 845C69E3
-P 625 2400
-F 0 "#GND010" H 625 2400 50  0001 C CNN
-F 1 "GND" H 525 2300 60  0000 L BNN
-F 2 "" H 625 2400 50  0001 C CNN
-F 3 "" H 625 2400 50  0001 C CNN
-	1    625  2400
-	1    0    0    -1
-$EndComp
-$Comp
 L Device:R R12
 U 1 1 5B546E94
@@
 $EndComp
 $Comp
+L Device:R R1
+U 1 1 4B3B8125
+P 7850 2100
+F 0 "R1" H 7700 2159 60  0000 L BNN
+F 1 "1k" H 7700 1970 60  0000 L BNN
+F 2 "Resistor_THT:R_Axial_DIN0207_L6.3mm_D2.5mm_P7.62mm_Horizontal" H 7850 2100 50  0001 C CNN
+F 3 "" H 7850 2100 50  0001 C CNN
+	1    7850 2100
+	1    0    0    1
+$EndComp
+$Comp
 L Device:R R6
 U 1 1 7A67179C
@@
 $EndComp
 $Comp
+L Device:R R5
+U 1 1 E15D264F
+P 9950 1300
+F 0 "R5" H 9900 1350 60  0000 L BNN
+F 1 "5k6" H 9800 1170 60  0000 L BNN
+F 2 "Resistor_THT:R_Axial_DIN0207_L6.3mm_D2.5mm_P7.62mm_Horizontal" H 9950 1300 50  0001 C CNN
+F 3 "" H 9950 1300 50  0001 C CNN
+	1    9950 1300
+	1    0    0    1
+$EndComp
+$Comp
+L Device:R R3
+U 1 1 83A6F2CB
+P 11350 3800
+F 0 "R3" H 11200 3859 60  0000 L BNN
+F 1 "470" H 11200 3670 60  0000 L BNN
+F 2 "Resistor_THT:R_Axial_DIN0207_L6.3mm_D2.5mm_P7.62mm_Horizontal" H 11350 3800 50  0001 C CNN
+F 3 "" H 11350 3800 50  0001 C CNN
+	1    11350 3800
+	1    0    0    -1
+$EndComp
+$Comp
+L Device:R R2
+U 1 1 70DE2412
+P 11350 4550
+F 0 "R2" H 11200 4609 60  0000 L BNN
+F 1 "5k6" H 11200 4420 60  0000 L BNN
+F 2 "Resistor_THT:R_Axial_DIN0207_L6.3mm_D2.5mm_P7.62mm_Horizontal" H 11350 4550 50  0001 C CNN
+F 3 "" H 11350 4550 50  0001 C CNN
+	1    11350 4550
+	1    0    0    -1
+$EndComp
+$Comp
 L Device:R R9
 U 1 1 5BA7DCB5
@@
 $EndComp
 $Comp
-L dos_5-0x-eagle-import:R-EU_0207_10 R1
-U 1 1 4B3B8125
-P 7850 2100
-F 0 "R1" H 7700 2159 60  0000 L BNN
-F 1 "1k" H 7700 1970 60  0000 L BNN
-F 2 "Resistor_THT:R_Axial_DIN0207_L6.3mm_D2.5mm_P7.62mm_Horizontal" H 7850 2100 50  0001 C CNN
-F 3 "" H 7850 2100 50  0001 C CNN
-	1    7850 2100
-	0    -1   1    0
-$EndComp
-$Comp
-L dos_5-0x-eagle-import:R-EU_0207_10 R5
-U 1 1 E15D264F
-P 9950 1300
-F 0 "R5" H 9900 1350 60  0000 L BNN
-F 1 "5k6" H 9800 1170 60  0000 L BNN
-F 2 "Resistor_THT:R_Axial_DIN0207_L6.3mm_D2.5mm_P7.62mm_Horizontal" H 9950 1300 50  0001 C CNN
-F 3 "" H 9950 1300 50  0001 C CNN
-	1    9950 1300
-	0    -1   1    0
-$EndComp
-$Comp
-L dos_5-0x-eagle-import:R-EU_0207_10 R3
-U 1 1 83A6F2CB
-P 11350 3800
-F 0 "R3" H 11200 3859 60  0000 L BNN
-F 1 "470" H 11200 3670 60  0000 L BNN
-F 2 "Resistor_THT:R_Axial_DIN0207_L6.3mm_D2.5mm_P7.62mm_Horizontal" H 11350 3800 50  0001 C CNN
-F 3 "" H 11350 3800 50  0001 C CNN
-	1    11350 3800
-	0    1    1    0
-$EndComp
-$Comp
-L dos_5-0x-eagle-import:R-EU_0207_10 R2
-U 1 1 70DE2412
-P 11350 4550
-F 0 "R2" H 11200 4609 60  0000 L BNN
-F 1 "5k6" H 11200 4420 60  0000 L BNN
-F 2 "Resistor_THT:R_Axial_DIN0207_L6.3mm_D2.5mm_P7.62mm_Horizontal" H 11350 4550 50  0001 C CNN
-F 3 "" H 11350 4550 50  0001 C CNN
-	1    11350 4550
-	0    1    1    0
-$EndComp
-$Comp
-L dos_5-0x-eagle-import:R-EU_0207_10 R22
+L Device:R R22
 U 1 1 5E8FC539
 P 22400 8450
@@
 F 3 "" H 22400 8450 50  0001 C CNN
 	1    22400 8450
-	0    1    1    0
+	1    0    0    -1
 $EndComp
 $Comp
-L dos_5-0x-eagle-import:R-EU_0207_10 R21
+L Device:R R21
 U 1 1 5F0584F0
 P 23750 8200
@@
 F 3 "" H 23750 8200 50  0001 C CNN
 	1    23750 8200
-	0    -1   -1   0
+	-1   0    0    1
 $EndComp
 $Comp
-L dos_5-0x-eagle-import:R-EU_0207_10 R18
+L Device:R R18
 U 1 1 5E8F296D
 P 25150 5100
@@
 F 3 "" H 25150 5100 50  0001 C CNN
 	1    25150 5100
-	0    -1   -1   0
+	-1   0    0    1
 $EndComp
 $Comp
@@
 $EndComp
 $Comp
-L dos_5-0x-eagle-import:C-EU025-030X050 C5
-U 1 1 F9108C4C
-P 9950 1700
-F 0 "C5" H 10010 1715 60  0000 L BNN
-F 1 "100n" H 10010 1515 60  0000 L BNN
-F 2 "Capacitor_THT:C_Disc_D5.0mm_W2.5mm_P5.00mm" H 9950 1700 50  0001 C CNN
-F 3 "" H 9950 1700 50  0001 C CNN
-	1    9950 1700
-	1    0    0    -1
-$EndComp
-$Comp
 L Device:C C1
 U 1 1 5BAD18CE
@@
 $EndComp
 $Comp
+L Device:C C5
+U 1 1 F9108C4C
+P 9950 1750
+F 0 "C5" H 10010 1765 60  0000 L BNN
+F 1 "100n" H 10010 1565 60  0000 L BNN
+F 2 "Capacitor_THT:C_Disc_D5.0mm_W2.5mm_P5.00mm" H 9950 1750 50  0001 C CNN
+F 3 "" H 9950 1750 50  0001 C CNN
+	1    9950 1750
+	1    0    0    -1
+$EndComp
+$Comp
 L Device:C C7
 U 1 1 5E518B43
@@
 $EndComp
 $Comp
-L ALEA:GAL22V10 U22
+L 8bits:GAL22V10 U22
 U 1 1 5E5B8A27
 P 11100 6100
@@
 $EndComp
 $Comp
-L ALEA:W27C512 U3
+L 8bits:W27C512 U3
 U 1 1 5E96589D
 P 5050 2750
@@
 $EndComp
 $Comp
-L ALEA:FDC_MB8877 U12
+L 8bits:FDC_MB8877 U12
 U 1 1 5E91CE08
 P 22250 6700
@@
 $EndComp
 $Comp
-L ALEA:ZX_Spectrum_Connector_GENERIC_SORTED J1
+L 8bits:ZX_Spectrum_Connector_GENERIC_SORTED J1
 U 1 1 5B1B7546
 P 2300 2750

Commit message: fix
Parts:
- removed Q1: BC639, Package_TO_SOT_THT:TO-92_Inline, symbol dos_5-0x-eagle-import:BC639
- added Q1: BC639, symbol Device:Q_NPN_ECB
- S1: symbol dos_5-0x-eagle-import:255SB -> beta128_r0.3-rescue:255SB-dos_5-0x-eagle-import
- S2: symbol dos_5-0x-eagle-import:10-XX -> beta128_r0.3-rescue:10-XX-dos_5-0x-eagle-import
Changed lines of the file:
@@
 	7650 2450 7650 2350
 Wire Wire Line
+	7725 3800 9250 3800
+Wire Wire Line
 	7850 1850 7850 1950
 Wire Wire Line
@@
 	8950 2750 8950 2800
 Wire Wire Line
-	9000 3800 9250 3800
-Wire Wire Line
 	9150 5500 9350 5500
 Wire Wire Line
@@
 	9400 3900 7150 3900
 Wire Wire Line
-	9400 4000 9000 4000
+	9400 4000 7725 4000
 Wire Wire Line
 	9400 4100 9350 4100
@@
 	14900 5600 15050 5600
 Wire Wire Line
-	15250 5300 15250 5400
-Wire Wire Line
-	15250 5800 15250 5900
-Wire Wire Line
-	15250 5900 15750 5900
+	15350 5350 15350 5400
+Wire Wire Line
+	15350 5800 15350 5900
+Wire Wire Line
+	15350 5900 15850 5900
 Wire Wire Line
 	17800 8200 17800 8550
@@
 	21850 3400 21850 3800
 Wire Wire Line
-	21850 3800 22100 3800
+	21850 3800 22425 3800
 Wire Wire Line
 	22000 3100 22200 3100
@@
 	22000 3500 22200 3500
 Wire Wire Line
-	22000 4000 22100 4000
-Wire Wire Line
-	22100 3900 21700 3900
+	22000 4000 22425 4000
 Wire Wire Line
 	22200 3100 22400 3100
@@
 	22400 8650 22350 8650
 Wire Wire Line
+	22425 3900 21700 3900
+Wire Wire Line
 	22750 5500 22850 5500
 Wire Wire Line
@@
 	22750 6000 22850 6000
 Wire Wire Line
-	22750 6300 22950 6300
-Wire Wire Line
-	22750 6400 22950 6400
-Wire Wire Line
-	22750 6500 22950 6500
-Wire Wire Line
-	22750 6600 22950 6600
+	22750 6300 23150 6300
+Wire Wire Line
+	22750 6400 23150 6400
+Wire Wire Line
+	22750 6500 23150 6500
+Wire Wire Line
+	22750 6600 23150 6600
 Wire Wire Line
 	22750 6700 22900 6700
@@
 	25950 3000 26100 3000
 Wire Wire Line
+	26000 5800 26650 5800
+Wire Wire Line
+	26000 5900 27350 5900
+Wire Wire Line
+	26000 6000 26850 6000
+Wire Wire Line
+	26000 6200 27350 6200
+Wire Wire Line
 	26200 8550 26400 8550
 Wire Wire Line
@@
 	26350 4100 26550 4100
 Wire Wire Line
-	26350 5800 26650 5800
-Wire Wire Line
-	26350 5900 27350 5900
-Wire Wire Line
-	26350 6000 26850 6000
-Wire Wire Line
-	26350 6200 27350 6200
-Wire Wire Line
 	26400 8550 26400 9050
 Wire Wire Line
@@
 	26400 9050 27350 9050
 Wire Wire Line
+	26425 6900 27350 6900
+Wire Wire Line
+	26425 7000 27350 7000
+Wire Wire Line
 	26450 3200 26700 3200
 Wire Wire Line
@@
 	26950 8850 27350 8850
 Wire Wire Line
+	27025 6000 27350 6000
+Wire Wire Line
 	27100 8700 27100 8750
 Wire Wire Line
 	27100 8750 27350 8750
 Wire Wire Line
-	27150 6000 27350 6000
-Wire Wire Line
-	27150 6900 27350 6900
-Wire Wire Line
-	27150 7000 27350 7000
-Wire Wire Line
 	27150 7100 27350 7100
 Wire Wire Line
@@
 	27300 3200 28650 3200
 Wire Wire Line
-	27300 4000 27850 4000
+	27300 4000 28150 4000
 Wire Wire Line
 	27300 8500 27300 8550
@@
 	27750 3550 28100 3550
 Wire Wire Line
-	27850 4400 27750 4400
+	27800 3450 28100 3450
 Wire Wire Line
 	27850 5700 27850 5800
@@
 	27850 9850 27850 9900
 Wire Wire Line
-	28050 3450 28100 3450
+	28150 4400 27750 4400
 Wire Wire Line
 	28350 8850 28500 8850
@@
 	28650 3450 28600 3450
 Wire Wire Line
-	28700 3550 28600 3550
+	29075 3550 28600 3550
 Wire Bus Line
 	3700 1000 3700 1600
@@
 	3700 3200 3700 3400
 Wire Bus Line
-	3700 3400 3700 3500
-Wire Bus Line
-	3700 3500 3700 3700
-Wire Bus Line
-	3700 3700 3700 3900
-Wire Bus Line
-	3700 3900 3700 4650
-Wire Bus Line
-	3700 4650 3700 4850
-Wire Bus Line
-	3700 4850 3700 4950
+	3700 3400 3700 3600
+Wire Bus Line
+	3700 3600 3700 3800
+Wire Bus Line
+	3700 3800 3700 4550
+Wire Bus Line
+	3700 4550 3700 4750
+Wire Bus Line
+	3700 4750 3700 4950
 Wire Bus Line
 	3700 4950 3700 5150
@@
 	5500 4850 5500 5050
 Wire Bus Line
-	5500 5050 5500 5250
-Wire Bus Line
-	5500 5250 5500 5600
-Wire Bus Line
-	6450 1000 6450 1150
-Wire Bus Line
-	6450 1150 6450 1600
-Wire Bus Line
-	6450 1600 6450 1700
+	5500 5050 5500 5150
+Wire Bus Line
+	5500 5150 5500 5600
+Wire Bus Line
+	6450 1000 6450 1500
+Wire Bus Line
+	6450 1500 6450 1700
 Wire Bus Line
 	6450 1700 6450 1900
@@
 	19750 4400 19750 4500
 Wire Bus Line
-	21250 6050 21250 6250
+	21250 5950 21250 6150
+Wire Bus Line
+	21250 6150 21250 6250
 Wire Bus Line
 	21250 6250 21250 6450
@@
 	21250 6650 21250 6750
 Wire Bus Line
-	21250 6750 21250 7350
+	21250 7150 21250 7350
 Text Notes 12800 5650 0    50   ~ 0
 ROM_CE = /(U8B_Q + A14 + A15 + /RD)
@@
 Text Label 8150 5200 0    50   ~ 0
 {slash}RESET
+Text Label 8225 4000 2    50   ~ 0
+{slash}A9
+Text Label 8250 3800 2    50   ~ 0
+{slash}(A14+A15)
 Text Label 9500 2450 0    50   ~ 0
 {slash}NMI
@@
 Text Label 10300 5900 2    50   ~ 0
 U8B_Q
+Text Label 12175 5900 2    50   ~ 0
+{slash}(A14+A15)
+Text Label 12175 6400 2    50   ~ 0
+{slash}A9
 Text Label 12850 4500 2    50   ~ 0
 U8B_Q
@@
 Text Label 14050 4650 0    50   ~ 0
 {slash}IORQ_EXT
-Text Label 15350 5900 0    50   ~ 0
+Text Label 15450 5900 0    50   ~ 0
 {slash}ROMCS
 Text Label 20000 4200 0    50   ~ 0
@@
 Text Label 20000 4300 0    50   ~ 0
 D'7
+Text Label 21250 6000 2    50   ~ 0
+D'[0...7]
+Text Label 21250 7200 2    50   ~ 0
+A[0...15]
 Text Label 21500 5950 0    50   ~ 0
 D'0
@@
 Text Label 21500 7250 0    50   ~ 0
 A6
+Text Label 22075 3900 0    50   ~ 0
+{slash}TR00
+Text Label 22100 3800 0    50   ~ 0
+{slash}WPRT
+Text Label 22100 4000 0    50   ~ 0
+{slash}IP
+Text Label 22925 6600 0    50   ~ 0
+{slash}WF
 Text Label 23200 3600 0    50   ~ 0
 D'3
@@
 Text Label 23200 4100 0    50   ~ 0
 D'6
+Text Label 23725 9550 0    50   ~ 0
+{slash}WF
+Text Label 26325 5800 2    50   ~ 0
+DS0
+Text Label 26325 5900 2    50   ~ 0
+DS3
+Text Label 26325 6000 2    50   ~ 0
+DS2
+Text Label 26325 6200 2    50   ~ 0
+DS1
 Text Label 26350 5700 2    50   ~ 0
 MOTOR_ON
+Text Label 27025 6900 0    50   ~ 0
+{slash}TR00
+Text Label 27025 7000 0    50   ~ 0
+{slash}WPRT
 Text Label 27100 6600 0    50   ~ 0
 STEP
+Text Label 27150 6000 0    50   ~ 0
+{slash}IP
 Text Label 27150 6500 0    50   ~ 0
 DIR
+Text Label 27975 4400 2    50   ~ 0
+DS3
+Text Label 28000 4000 2    50   ~ 0
+DS2
+Text Label 28050 3450 2    50   ~ 0
+DS0
+Text Label 28925 3550 2    50   ~ 0
+DS1
 Text GLabel 850  1800 0    50   Input ~ 0
 plus3_5V
@@
 Text GLabel 8250 2450 0    50   Input ~ 0
 A14+A15
-Text GLabel 9000 3800 0    50   Input ~ 0
-{slash}(A14+A15)
-Text GLabel 9000 4000 0    50   Input ~ 0
-{slash}A9
 Text GLabel 12350 5600 2    50   Output ~ 0
 {slash}ROM_CE
@@
 Text GLabel 12350 5800 2    50   Output ~ 0
 DIR
-Text GLabel 12350 5900 2    50   Output ~ 0
-{slash}(A14+A15)
 Text GLabel 12350 6000 2    50   Output ~ 0
 A14+A15
@@
 Text GLabel 12350 6300 2    50   Output ~ 0
 U11_OEB
-Text GLabel 12350 6400 2    50   Output ~ 0
-{slash}A9
 Text GLabel 12350 6500 2    50   Output ~ 0
 IO_WR1
@@
 Text GLabel 21750 4600 2    50   Input ~ 0
 U11_OEB
-Text GLabel 22100 3800 2    50   Input ~ 0
-{slash}WPRT
-Text GLabel 22100 3900 2    50   Input ~ 0
-{slash}TR00
-Text GLabel 22100 4000 2    50   Input ~ 0
-{slash}IP
 Text GLabel 22100 4200 2    50   Input ~ 0
 DRQ
@@
 Text GLabel 22850 6000 2    50   Input ~ 0
 FD_CLK
-Text GLabel 22950 6300 2    50   Input ~ 0
-FDC_WPRT
-Text GLabel 22950 6400 2    50   Input ~ 0
-FDC_IP
-Text GLabel 22950 6500 2    50   Input ~ 0
-FDC_TR00
-Text GLabel 22950 6600 2    50   Input ~ 0
-{slash}WF
 Text GLabel 23050 7600 2    50   Input ~ 0
 HLT
 Text GLabel 23150 4300 0    50   Input ~ 0
 U10_CP
+Text GLabel 23150 6300 2    50   Input ~ 0
+FDC_WPRT
+Text GLabel 23150 6400 2    50   Input ~ 0
+FDC_IP
+Text GLabel 23150 6500 2    50   Input ~ 0
+FDC_TR00
 Text GLabel 23650 8450 0    50   Input ~ 0
 DATA_READ
 Text GLabel 23650 9350 0    50   Input ~ 0
 4Mhz
-Text GLabel 23650 9550 0    50   Input ~ 0
-{slash}WF
 Text GLabel 24600 3600 2    50   Input ~ 0
 HLT
@@
 Text GLabel 26100 3000 2    50   Output ~ 0
 HEAD
-Text GLabel 26350 5800 0    50   Input ~ 0
-DS0
-Text GLabel 26350 5900 0    50   Input ~ 0
-DS3
-Text GLabel 26350 6000 0    50   Input ~ 0
-DS2
-Text GLabel 26350 6200 0    50   Input ~ 0
-DS1
 Text GLabel 26500 8550 2    50   Output ~ 0
 FD_DATA
-Text GLabel 27150 6000 0    50   Input ~ 0
-{slash}IP
-Text GLabel 27150 6900 0    50   Output ~ 0
-{slash}TR00
-Text GLabel 27150 7000 0    50   Output ~ 0
-{slash}WPRT
-Text GLabel 27150 7100 0    50   Output ~ 0
+Text GLabel 27150 7100 0    50   Input ~ 0
 DATA_READ
 Text GLabel 27150 7200 0    50   Input ~ 0
 HEAD
-Text GLabel 27850 4000 2    50   Output ~ 0
-DS2
-Text GLabel 27850 4400 2    50   Output ~ 0
-DS3
-Text GLabel 28050 3450 0    50   Output ~ 0
-DS0
 Text GLabel 28550 8850 2    50   Output ~ 0
 FD_CLK
-Text GLabel 28700 3550 2    50   Output ~ 0
-DS1
 $Comp
 L power:PWR_FLAG #FLG0102
@@
 L power:+5V #PWR0109
 U 1 1 5F93A25A
-P 15250 5300
-F 0 "#PWR0109" H 15250 5150 50  0001 C CNN
-F 1 "+5V" H 15265 5473 50  0000 C CNN
-F 2 "" H 15250 5300 50  0001 C CNN
-F 3 "" H 15250 5300 50  0001 C CNN
-	1    15250 5300
+P 15350 5350
+F 0 "#PWR0109" H 15350 5200 50  0001 C CNN
+F 1 "+5V" H 15365 5523 50  0000 C CNN
+F 2 "" H 15350 5350 50  0001 C CNN
+F 3 "" H 15350 5350 50  0001 C CNN
+	1    15350 5350
 	1    0    0    -1
 $EndComp
@@
 $EndComp
 $Comp
-L dos_5-0x-eagle-import:BC639 Q1
-U 1 1 7A211019
-P 15150 5600
-F 0 "Q1" H 15350 5700 60  0000 L BNN
-F 1 "BC639" H 15350 5600 60  0000 L BNN
-F 2 "Package_TO_SOT_THT:TO-92_Inline" H 15150 5600 50  0001 C CNN
-F 3 "" H 15150 5600 50  0001 C CNN
-	1    15150 5600
-	1    0    0    -1
-$EndComp
-$Comp
 L Connector:Conn_01x05_Male JP5
 U 1 1 5E518CE8
@@
 $EndComp
 $Comp
-L dos_5-0x-eagle-import:10-XX S2
+L beta128_r0.3-rescue:10-XX-dos_5-0x-eagle-import S2
 U 1 1 F82F9BF5
 P 7350 2350
@@
 $EndComp
 $Comp
-L dos_5-0x-eagle-import:255SB S1
+L beta128_r0.3-rescue:255SB-dos_5-0x-eagle-import S1
 U 1 1 CEBFFD5E
 P 12100 3200
@@
 $EndComp
 $Comp
+L Device:Q_NPN_ECB Q1
+U 1 1 5E723837
+P 15250 5600
+F 0 "Q1" H 15441 5645 50  0000 L CNN
+F 1 "BC639" H 15441 5555 50  0000 L CNN
+F 2 "" H 15450 5700 50  0001 C CNN
+F 3 "~" H 15250 5600 50  0001 C CNN
+	1    15250 5600
+	1    0    0    -1
+$EndComp
+$Comp
